File: feather/burrboard.kicad_sch (KiCad schematic)
At the start: 30 parts, among them J1 J1, J2 J2, J3 Conn_01x02_Male, U1 TMP36, U2 ADXL345BCCZ

Commit message: Final fixes
Parts:
- gave numbers to parts that had none: 1
Changed lines of the file:
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@@
   (symbol (lib_id "burrboard:TEMT6000X01") (at 177.8 43.18 90) (unit 1)
     (in_bom yes) (on_board yes) (fields_autoplaced)
-    (property "Reference" "Q?" (id 0) (at 184.15 30.4799 90)
+    (property "Reference" "Q1" (id 0) (at 184.15 30.4799 90)
       (effects (font (size 1.27 1.27)) (justify right))
     )
@@
     )
     (path "/666dc925-2b95-4de4-a148-45e51fb4be3f"
-      (reference "Q?") (unit 1) (value "TEMT6000X01") (footprint "burrboard:Phototransistor_SMD_4x2mm_TEMT6000X01")
+      (reference "Q1") (unit 1) (value "TEMT6000X01") (footprint "burrboard:Phototransistor_SMD_4x2mm_TEMT6000X01")
     )
     (path "/00000000-0000-0000-0000-000061c212d9"

Commit message: Add missing names
Parts:
- C5: MPN Vishay Vitramon -> VJ0805A100JXAAC; Manufacturer Samsung Electro-Mechanics -> Vishay Vitramon
Changed lines of the file:
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@@
       (effects (font (size 1.27 1.27)) hide)
     )
-    (property "MPN" "Vishay Vitramon" (id 5) (at 139.7 52.07 0)
+    (property "MPN" "VJ0805A100JXAAC" (id 5) (at 139.7 52.07 0)
       (effects (font (size 1.27 1.27)) hide)
     )
-    (property "Manufacturer" "Samsung Electro-Mechanics" (id 6) (at 139.7 52.07 0)
+    (property "Manufacturer" "Vishay Vitramon" (id 6) (at 139.7 52.07 0)
       (effects (font (size 1.27 1.27)) hide)
     )
