File: hardware/feather/kicad/burrboard.kicad_pcb (KiCad board)
At the start: 2 copper layers, 50.8 x 81.3 mm, 31 parts, among them J1 J1, J2 J2, J3 SWD, J4 SWDCLK, J5 SWDIO, Q1 TEMT6000X01, U1 TMP36

Commit message: Updated
Parts:
- removed J3: SWD, Connector_PinHeader_2.54mm:PinHeader_1x04_P2.54mm_Vertical
- removed J4: SWDCLK, TestPoint:TestPoint_THTPad_D1.0mm_Drill0.5mm
- removed J5: SWDIO, TestPoint:TestPoint_THTPad_D1.0mm_Drill0.5mm
- added C2: 10u, Capacitor_SMD:C_0805_2012Metric, F.Cu at (202.9, 72.1)
- added C3: 100n, Capacitor_SMD:C_0805_2012Metric, F.Cu at (204.0, 68.8)
- added C4: 100n, Capacitor_SMD:C_0805_2012Metric, F.Cu at (203.7, 75.9)
- added R3: 10k, Resistor_SMD:R_0805_2012Metric, F.Cu at (219.5, 75.9)
- added R9: 10k, Resistor_SMD:R_0805_2012Metric, F.Cu at (219.7, 70.9)
- added U2: ADXL345BCCZ, burrboard:LGA-14_3x5mm_RevA, F.Cu at (209.6, 72.4)
Connections:
- J2 pad 1: unconnected-(J2-Pad1) -> /SDA
- J2 pad 2: unconnected-(J2-Pad2) -> /SCL
- J2 pad 8: unconnected-(J2-Pad8) -> /F5
- Q1 pad 3: /F1 -> /F0
- R4 pad 1: /F4 -> /F5
- R5 pad 1: /F3 -> /F4
- R8 pad 2: /F2 -> /F3
- S1 pad 1: /F4 -> /F5
- S2 pad 1: /F3 -> /F4
Routing:
- net /F5: track 0.00 -> 79.8 mm, vias 0 -> 1
- net /F0: track 85.0 -> 157.6 mm, vias 1 -> 5
- net /F3: track 85.0 -> 40.4 mm
- net /F1: track 47.1 -> 20.3 mm
- net Net-(J3-Pad3): track 25.6 -> 0.00 mm, vias 1 -> 0
- net /SDA: track 0.00 -> 24.2 mm
- net Net-(J3-Pad2): track 23.9 -> 0.00 mm
- net /SCL: track 0.00 -> 14.9 mm
- net /3V3: track 122.7 -> 109.1 mm
- net /F2: track 31.2 -> 18.5 mm, vias 0 -> 1
- net /F4: track 78.9 -> 86.1 mm, vias 2 -> 1
- net GND: vias 6 -> 8
