File: hardware/feather/burrboard.kicad_sch (KiCad schematic)
At the start: 27 parts, among them J1 J1, J2 J2, J3 SWD, J4 SWDCLK, J5 SWDIO, Q1 TEMT6000X01, U1 TMP36

Commit message: Fixup
Parts:
- removed D5: SD103ATW, Package_TO_SOT_SMD:SOT-363_SC-70-6, symbol Diode:SD103ATW
- added D5: NRVB0540T3G, SOD3716X135N, symbol schottky2:NRVB0540T3G
- J3: Manufacturer (none) -> TE Connectivity AMP Connectors
- J4, J5: Manufacturer (none) -> Mill-Max Manufacturing Corp.
- Q1: Manufacturer (none) -> Vishay; Manufacturer_Name Vishay -> (none)
Connections:
- net VDD: now also D5.2
- net at S3.2 (B): now also D5.1
Other:
- moved on the sheet: S3

Commit message: Rev 3.5
Parts:
- removed J3: SWD, Connector_PinHeader_2.54mm:PinHeader_1x04_P2.54mm_Vertical, symbol Connector:Conn_01x04_Male
- removed J4: SWDCLK, TestPoint:TestPoint_THTPad_D1.0mm_Drill0.5mm, symbol Connector:Conn_01x01_Male
- removed J5: SWDIO, TestPoint:TestPoint_THTPad_D1.0mm_Drill0.5mm, symbol Connector:Conn_01x01_Male
- added C2: 10u, Capacitor_SMD:C_0805_2012Metric, symbol Device:C
- added C3, C4: 100n, Capacitor_SMD:C_0805_2012Metric, symbol Device:C
- added R3, R9: 10k, Resistor_SMD:R_0805_2012Metric, symbol Device:R
- added U2: ADXL345BCCZ, burrboard:LGA-14_3x5mm_RevA, symbol burrboard:ADXL345BCCZ
- D5: footprint SOD3716X135N -> schottky2:SOD3716X135N
Connections:
- net F0: now also Q1.3 (C), C2.1, C3.1, C4.1, R3.2, R9.2, U2.1 (VDD_I/O), U2.6 (VS), U2.7 (~{CS})
- net F1: now also U2.8 (INT1); no longer Q1.3 (C)
- net F2: now also U2.9 (INT2); no longer R8.2
- net F3: now also R8.2; no longer R5.1, S2.1
- net F4: now also R5.1, S2.1; no longer R4.1, S1.1
- net GND: now also C2.2, C3.2, C4.2, U2.12 (SDO/ALT_ADD), U2.2 (GND), U2.4 (GND), U2.5 (GND)
- net SDA: now reaches J2.1 (Pin_1)
- net SDA: now also R3.1, U2.13 (SDA/SDI/SDIO)
- net SCL: now reaches J2.2 (Pin_2)
- net SCL: now also R9.1, U2.14 (SCL/SCLK)
- net F5: now reaches J2.8 (Pin_8)
- net F5: now also R4.1, S1.1
- no-connect marks 20 -> 19

Commit message: Rev 4
Parts:
- added J3: SWD, Connector_PinHeader_2.54mm:PinHeader_1x04_P2.54mm_Vertical, symbol Connector:Conn_01x04_Male
- added J4: SWDCLK, TestPoint:TestPoint_THTPad_D1.0mm_Drill0.5mm, symbol Connector:Conn_01x01_Male
- added J5: SWDIO, TestPoint:TestPoint_THTPad_D1.0mm_Drill0.5mm, symbol Connector:Conn_01x01_Male
Connections:
- net 3V3: now also J3.1 (Pin_1)
- net GND: now also J3.4 (Pin_4)
- new net: J3.3 (Pin_3), J5.1 (Pin_1)
- new net: J3.2 (Pin_2), J4.1 (Pin_1)
Other:
- note added: "Accelerometer"
- note added: "Debug"
- moved on the sheet: C2, C3, C4, R3, R9, U2

Commit message: Increase size of pogopin footprint
Parts:
- J3: now left out of the parts list
- J4, J5: footprint TestPoint:TestPoint_THTPad_D1.0mm_Drill0.5mm -> TestPoint:TestPoint_THTPad_D1.5mm_Drill0.7mm; now left out of the parts list
Changed lines of the file:
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@@
   )
   (symbol (lib_id "Connector:Conn_01x01_Male") (at 72.39 185.674 180) (unit 1)
-    (in_bom yes) (on_board yes)
+    (in_bom no) (on_board yes)
     (property "Reference" "J5" (id 0) (at 69.596 188.214 0))
     (property "Value" "SWDIO" (id 1) (at 76.2 185.674 0))
-    (property "Footprint" "TestPoint:TestPoint_THTPad_D1.0mm_Drill0.5mm" (id 2) (at 72.39 185.674 0)
+    (property "Footprint" "TestPoint:TestPoint_THTPad_D1.5mm_Drill0.7mm" (id 2) (at 72.39 185.674 0)
       (effects (font (size 1.27 1.27)) hide)
     )
@@
   )
   (symbol (lib_id "Connector:Conn_01x04_Male") (at 41.402 183.134 0) (unit 1)
-    (in_bom yes) (on_board yes) (fields_autoplaced)
+    (in_bom no) (on_board yes) (fields_autoplaced)
     (property "Reference" "J3" (id 0) (at 42.037 175.768 0))
     (property "Value" "SWD" (id 1) (at 42.037 178.308 0))
@@
   )
   (symbol (lib_id "Connector:Conn_01x01_Male") (at 72.39 183.134 180) (unit 1)
-    (in_bom yes) (on_board yes)
+    (in_bom no) (on_board yes)
     (property "Reference" "J4" (id 0) (at 69.596 179.832 0))
     (property "Value" "SWDCLK" (id 1) (at 76.962 183.134 0))
-    (property "Footprint" "TestPoint:TestPoint_THTPad_D1.0mm_Drill0.5mm" (id 2) (at 72.39 183.134 0)
+    (property "Footprint" "TestPoint:TestPoint_THTPad_D1.5mm_Drill0.7mm" (id 2) (at 72.39 183.134 0)
       (effects (font (size 1.27 1.27)) hide)
     )
@@
     )
     (path "/d063ba46-22f6-4e50-9d5e-95f13fbaf268"
-      (reference "J4") (unit 1) (value "SWDCLK") (footprint "TestPoint:TestPoint_THTPad_D1.0mm_Drill0.5mm")
+      (reference "J4") (unit 1) (value "SWDCLK") (footprint "TestPoint:TestPoint_THTPad_D1.5mm_Drill0.7mm")
     )
     (path "/cba8ab97-0377-43bd-bef7-6314ce99d4ae"
-      (reference "J5") (unit 1) (value "SWDIO") (footprint "TestPoint:TestPoint_THTPad_D1.0mm_Drill0.5mm")
+      (reference "J5") (unit 1) (value "SWDIO") (footprint "TestPoint:TestPoint_THTPad_D1.5mm_Drill0.7mm")
     )
     (path "/666dc925-2b95-4de4-a148-45e51fb4be3f"

Commit message: Make rev 3.5 final version
Parts:
- removed J3: SWD, Connector_PinHeader_2.54mm:PinHeader_1x04_P2.54mm_Vertical, symbol Connector:Conn_01x04_Male
- removed J4: SWDCLK, TestPoint:TestPoint_THTPad_D1.5mm_Drill0.7mm, symbol Connector:Conn_01x01_Male
- removed J5: SWDIO, TestPoint:TestPoint_THTPad_D1.5mm_Drill0.7mm, symbol Connector:Conn_01x01_Male
Other:
- note removed: "Accelerometer"
- note removed: "Debug"
- moved on the sheet: C2, C3, C4, R3, R9, U2
