File: hardware/feather/burrboard.kicad_sch (KiCad schematic)
At the start: 30 parts, among them J1 J1, J2 J2, Q1 TEMT6000X01, U1 TMP36, U2 ADXL345BCCZ

Commit message: Update component
Parts:
- D5: value NRVB0540T3G -> CDBW0540-G; Arrow Part Number NRVB0540T3G -> (none); Arrow Price/Stock https://www.arrow.com/en/products/nrvb0540t3g/on-semiconduc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 -> (none); Digi-Key_PN NRVB0540T3GOSTR-ND -> 641-1327-2-ND; Height 1.35 -> (none); MPN NRVB0540T3G -> CDBW0540-G; Manufacturer ON Semiconductor -> Comchip Technology; Mouser Part Number 863-NRVB0540T3G -> (none); Mouser Price/Stock https://www.mouser.co.uk/ProductDetail/onsemi/NRVB0540T3G?q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 -> (none)
Changed lines of the file:
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@@
     (in_bom yes) (on_board yes) (fields_autoplaced)
     (property "Reference" "D5" (id 0) (at 141.224 155.956 0))
-    (property "Value" "NRVB0540T3G" (id 1) (at 141.224 158.496 0))
+    (property "Value" "CDBW0540-G" (id 1) (at 141.224 158.496 0))
     (property "Footprint" "schottky2:SOD3716X135N" (id 2) (at 138.684 167.386 0)
       (effects (font (size 1.27 1.27)) (justify left) hide)
     )
-    (property "Datasheet" "https://www.mouser.de/datasheet/2/308/MBR0540T1_D-1810841.pdf" (id 3) (at 138.684 164.846 0)
+    (property "Datasheet" "https://www.comchiptech.com/admin/files/product/CDBW0520L-HF%20Thru824572.%20CDBW0540-HF%20RevA.pdf" (id 3) (at 138.684 164.846 0)
       (effects (font (size 1.27 1.27)) (justify left) hide)
     )
@@
       (effects (font (size 1.27 1.27)) (justify left) hide)
     )
-    (property "Height" "1.35" (id 5) (at 138.684 159.766 0)
-      (effects (font (size 1.27 1.27)) (justify left) hide)
-    )
-    (property "Manufacturer" "ON Semiconductor" (id 6) (at 138.684 157.226 0)
-      (effects (font (size 1.27 1.27)) (justify left) hide)
-    )
-    (property "MPN" "NRVB0540T3G" (id 7) (at 138.684 154.686 0)
-      (effects (font (size 1.27 1.27)) (justify left) hide)
-    )
-    (property "Mouser Part Number" "863-NRVB0540T3G" (id 8) (at 138.684 152.146 0)
-      (effects (font (size 1.27 1.27)) (justify left) hide)
-    )
-    (property "Mouser Price/Stock" "https://www.mouser.co.uk/ProductDetail/onsemi/NRVB0540T3G?qs=JZRcihQa5bv2BoZB9hCl7w%3D%3D" (id 9) (at 138.684 149.606 0)
-      (effects (font (size 1.27 1.27)) (justify left) hide)
-    )
-    (property "Arrow Part Number" "NRVB0540T3G" (id 10) (at 138.684 147.066 0)
-      (effects (font (size 1.27 1.27)) (justify left) hide)
-    )
-    (property "Arrow Price/Stock" "https://www.arrow.com/en/products/nrvb0540t3g/on-semiconductor" (id 11) (at 138.684 144.526 0)
-      (effects (font (size 1.27 1.27)) (justify left) hide)
-    )
-    (property "Digi-Key_PN" "NRVB0540T3GOSTR-ND" (id 12) (at 151.384 163.576 0)
+    (property "Manufacturer" "Comchip Technology" (id 6) (at 138.684 157.226 0)
+      (effects (font (size 1.27 1.27)) (justify left) hide)
+    )
+    (property "MPN" "CDBW0540-G" (id 7) (at 138.684 154.686 0)
+      (effects (font (size 1.27 1.27)) (justify left) hide)
+    )
+    (property "Digi-Key_PN" "641-1327-2-ND" (id 12) (at 151.384 163.576 0)
       (effects (font (size 1.27 1.27)) hide)
     )
@@
     )
     (path "/232fab35-17b2-4202-aa20-97192fb94a6a"
-      (reference "D5") (unit 1) (value "NRVB0540T3G") (footprint "schottky2:SOD3716X135N")
+      (reference "D5") (unit 1) (value "CDBW0540-G") (footprint "schottky2:SOD3716X135N")
     )
     (path "/00000000-0000-0000-0000-00005d375c76"
